Commit message: Changed the position of the sensor

File: basics_turtlebot/turtlebot_description/urdf/turtlebot_properties.urdf.xacro (robot description, xacro)
@@ -19,7 +19,8 @@
      (currently in development and awaiting feedback)
    -->
-	<xacro:property name="cam_px" value="-0.087" />
+	<!-- <xacro:property name="cam_px" value="-0.087" /> -->
+  <xacro:property name="cam_px" value="0.115" />
 <!--	<xacro:property name="cam_py" value="-0.0125" /> Y varies for different configurations. get sets in sensors_urdf -->
-	<xacro:property name="cam_pz" value="0.2870" />
+	<xacro:property name="cam_pz" value="0.21" />
 	<xacro:property name="cam_or" value="0" />
 	<xacro:property name="cam_op" value="0" />

Commit message: First measurement - different sensor location of the Xtion pro (seems to be incorrect when running gmapping)

File: basics_turtlebot/turtlebot_description/urdf/turtlebot_properties.urdf.xacro (robot description, xacro)
@@ -20,7 +20,7 @@
    -->
 	<!-- <xacro:property name="cam_px" value="-0.087" /> -->
-  <xacro:property name="cam_px" value="0.115" />
+  <xacro:property name="cam_px" value="-0.105" />
 <!--	<xacro:property name="cam_py" value="-0.0125" /> Y varies for different configurations. get sets in sensors_urdf -->
-	<xacro:property name="cam_pz" value="0.21" />
+	<xacro:property name="cam_pz" value="0.28" />
 	<xacro:property name="cam_or" value="0" />
 	<xacro:property name="cam_op" value="0" />

Commit message: The sensor placement values did not seem to be correct.

File: basics_turtlebot/turtlebot_description/urdf/turtlebot_properties.urdf.xacro (robot description, xacro)
@@ -20,7 +20,7 @@
    -->
 	<!-- <xacro:property name="cam_px" value="-0.087" /> -->
-  <xacro:property name="cam_px" value="-0.105" />
+  <xacro:property name="cam_px" value="-0.095" />
 <!--	<xacro:property name="cam_py" value="-0.0125" /> Y varies for different configurations. get sets in sensors_urdf -->
-	<xacro:property name="cam_pz" value="0.28" />
+	<xacro:property name="cam_pz" value="0.29" />
 	<xacro:property name="cam_or" value="0" />
 	<xacro:property name="cam_op" value="0" />

Commit message: Adjusted the sensor values back to default, as the kinect is remounted

File: basics_turtlebot/turtlebot_description/urdf/turtlebot_properties.urdf.xacro (robot description, xacro)
@@ -20,9 +20,9 @@
    -->
 	<!-- <xacro:property name="cam_px" value="-0.087" /> -->
-  <xacro:property name="cam_px" value="-0.095" />
-<!--	<xacro:property name="cam_py" value="-0.0125" /> Y varies for different configurations. get sets in sensors_urdf -->
-	<xacro:property name="cam_pz" value="0.29" />
+  <xacro:property name="cam_px" value="-0.087" />
+  <!--	<xacro:property name="cam_py" value="-0.0125" /> Y varies for different configurations. get sets in sensors_urdf -->
+	<xacro:property name="cam_pz" value="0.2870" />
 	<xacro:property name="cam_or" value="0" />
 	<xacro:property name="cam_op" value="0" />
-	<xacro:property name="cam_oy" value="0" />
+  <xacro:property name="cam_oy" value="0" />
 </robot>
